Commit message: making the hfe joint not continuous otherwise we have issues with pinocchio

File: aliengo_description/urdfs/const.xacro (robot description, xacro)
@@ -35,4 +35,6 @@
     <xacro:property name="hip_velocity_max" value="20"/>
     <xacro:property name="hip_torque_max" value="44"/>
+    <xacro:property name="upperleg_position_max" value="${PI}"/>
+    <xacro:property name="upperleg_position_min" value="${-PI}"/>
     <xacro:property name="upperleg_velocity_max" value="20"/>
     <xacro:property name="upperleg_torque_max" value="44"/>

File: aliengo_description/urdfs/leg.xacro (robot description, xacro)
@@ -63,5 +63,5 @@
             </collision>
         </link> -->
-        <joint name="${name}_hfe_joint" type="continuous">
+        <joint name="${name}_hfe_joint" type="revolute">
             <origin rpy="0 0 0" xyz="0 ${upperleg_offset*mirror} 0"/>
             <parent link="${name}_hip"/>
@@ -69,5 +69,5 @@
             <axis xyz="0 1 0"/>
             <dynamics damping="${damping}" friction="${friction}"/>
-            <limit effort="${upperleg_torque_max}" velocity="${upperleg_velocity_max}"/>
+            <limit effort="${upperleg_torque_max}" velocity="${upperleg_velocity_max}"  lower="${upperleg_position_min}" upper="${upperleg_position_max}"/>
         </joint>
         <link name="${name}_upperleg">
