Commit message: changing go0 from sdrf

File: aliengo_description/robots/aliengo.srdf.xacro (robot description, xacro)
@@ -50,30 +50,16 @@
     </group>
     <group_state group="chains" name="standup">
-        <joint name="lf_haa_joint" value="0.1"/>
-        <joint name="lf_hfe_joint" value="0.67"/>
-        <joint name="lf_kfe_joint" value="-1.3"/>
-        <joint name="rf_haa_joint" value="-0.1"/>
-        <joint name="rf_hfe_joint" value="0.67"/>
-        <joint name="rf_kfe_joint" value="-1.3"/>
-        <joint name="lh_haa_joint" value="0.1"/>
-        <joint name="lh_hfe_joint" value="0.67"/>
-        <joint name="lh_kfe_joint" value="-1.3"/>
-        <joint name="rh_haa_joint" value="-0.1"/>
-        <joint name="rh_hfe_joint" value="0.67"/>
-        <joint name="rh_kfe_joint" value="-1.3"/>
-    </group_state>
-    <group_state group="chains" name="standdown">
-        <joint name="lf_haa_joint" value="0.60"/>
-        <joint name="lf_hfe_joint" value="1.70"/>
-        <joint name="lf_kfe_joint" value="-2.77"/>
-        <joint name="rf_haa_joint" value="-0.60"/>
-        <joint name="rf_hfe_joint" value="1.70"/>
-        <joint name="rf_kfe_joint" value="-2.77"/>
-        <joint name="lh_haa_joint" value="0.60"/>
-        <joint name="lh_hfe_joint" value="1.52"/>
-        <joint name="lh_kfe_joint" value="-2.77"/>
-        <joint name="rh_haa_joint" value="-0.60"/>
-        <joint name="rh_hfe_joint" value="1.52"/>
-        <joint name="rh_kfe_joint" value="-2.77"/>
+        <joint name="lf_haa_joint" value="0.2"/>
+        <joint name="lf_hfe_joint" value="0.7"/>
+        <joint name="lf_kfe_joint" value="-14"/>
+        <joint name="rf_haa_joint" value="-0.2"/>
+        <joint name="rf_hfe_joint" value="0.7"/>
+        <joint name="rf_kfe_joint" value="-1.4"/>
+        <joint name="lh_haa_joint" value="0.2"/>
+        <joint name="lh_hfe_joint" value="0.7"/>
+        <joint name="lh_kfe_joint" value="-1.4"/>
+        <joint name="rh_haa_joint" value="-0.2"/>
+        <joint name="rh_hfe_joint" value="0.7"/>
+        <joint name="rh_kfe_joint" value="-1.4"/>
     </group_state>
 </robot>
