Commit message: bugfix: missing base link joint, the tf tree is no longer cut

File: aliengo_description/robots/aliengo.urdf.xacro (robot description, xacro)
@@ -31,7 +31,13 @@
               <origin rpy="0 0 0" xyz="0 0 0"/>
               <parent link="world"/>
-              <child link="trunk"/>
+              <child link="base_link"/>
             </joint>
     </xacro:if>
+    <link name="base_link" />
+   <joint name="floating_base" type="fixed">
+    <origin rpy="0 0 0" xyz="0 0 0"/>
+    <parent link="base_link"/>
+    <child link="trunk"/>
+   </joint>
     <link name="trunk">
         <visual>
